File: schematics/kicad/teensy41_fpga_theremin/teensy41_fpga_theremin.kicad_pcb (KiCad board)
At the start: 2 copper layers, 199.4 x 61 mm, 52 parts, among them J1 Volume Sensor, J10 Ground, J2 Pitch Sensor, J3 Power In +5V, J4 EXPR PED 1, J6 LINE IN, J7 LINE OUT, J8 Pitch Pgm, J9 Vol Pgm, U1 Teensy41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

Commit message: teensy fpga theremin main pcb
Parts:
- added C18: 10uF, Capacitor_SMD:C_0805_2012Metric, F.Cu at (77.5, 123.2)
- added C27: 10uF, Capacitor_SMD:C_0805_2012Metric, F.Cu at (81.9, 123.2)
- added C28: 10uF, Capacitor_SMD:C_0805_2012Metric, F.Cu at (86.4, 123.2)
- added C29: 2.2uF, Capacitor_SMD:C_0805_2012Metric, F.Cu at (78.7, 111.8)
- added C30: 2.2uF, Capacitor_SMD:C_0805_2012Metric, F.Cu at (205.7, 59.7)
- added C31: 10nF, Capacitor_SMD:C_0805_2012Metric, F.Cu at (78.7, 108.0)
- added C32: 10nF, Capacitor_SMD:C_0805_2012Metric, F.Cu at (205.7, 62.2)
- added C33: 10uF, Capacitor_SMD:C_0805_2012Metric, F.Cu at (69.8, 109.2)
- added C34: 10uF, Capacitor_SMD:C_0805_2012Metric, F.Cu at (213.4, 61.3)
- added D2: STPS1L30A, Diode_SMD:D_SMA, F.Cu at (99.6, 140.4)
- added D3: STPS1L30A, Diode_SMD:D_SMA, F.Cu at (99.6, 145.0)
- added D4: STPS1L30A, Diode_SMD:D_SMA, F.Cu at (99.6, 149.5)
- added D5: STPS1L30A, Diode_SMD:D_SMA, F.Cu at (99.6, 154.1)
- added J11: PREF_VCC, Connector_PinHeader_2.54mm:PinHeader_2x02_P2.54mm_Vertical, F.Cu at (218.4, 67.3)
- added J12: PSNS_VCC, Connector_PinHeader_2.54mm:PinHeader_2x03_P2.54mm_Vertical, F.Cu at (218.4, 57.1)
- added J13: VDRV_VCC, Connector_PinHeader_2.54mm:PinHeader_2x03_P2.54mm_Vertical, F.Cu at (64.8, 95.2)
- added J14: VREF_VCC, Connector_PinHeader_2.54mm:PinHeader_2x02_P2.54mm_Vertical, F.Cu at (64.8, 102.9)
- added J15: VSNS_VCC, Connector_PinHeader_2.54mm:PinHeader_2x03_P2.54mm_Vertical, F.Cu at (64.8, 113.0)
- added J5: PDRV_VCC, Connector_PinHeader_2.54mm:PinHeader_2x03_P2.54mm_Vertical, F.Cu at (218.4, 74.9)
- added U11: LD3985G33R_TSOT23, Package_TO_SOT_SMD:TSOT-23-5, F.Cu at (73.7, 109.2)
- added U12: LD3985G33R_TSOT23, Package_TO_SOT_SMD:TSOT-23-5, F.Cu at (209.6, 61.0)
- J2: value Pitch Sensor -> Conn_02x06_Odd_Even
- moved D1 66.5 mm to (99.6, 135.9)
- moved C1 30.5 mm to (100.3, 76.5)
- moved C7 30.5 mm to (104.1, 76.2)
- moved FB1 30.5 mm to (102.0, 71.1)
- moved C10 14.8 mm to (77.5, 100.3), turned to 0 degrees
- moved C4 13.7 mm to (77.8, 102.9)
- moved C24 13.7 mm to (69.8, 101.3)
- moved U8 13.7 mm to (73.7, 101.6)
- moved C2 13.5 mm to (196.8, 58.4)
- moved C8 13.5 mm to (191.8, 58.4)
- moved FB2 13.5 mm to (194.3, 63.5)
- moved J1 12.5 mm to (49.5, 96.5)
- moved J2 9.16 mm to (233.7, 73.7)
- moved C3 8.52 mm to (77.8, 95.2)
- moved C5 8.36 mm to (205.4, 67.3)
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Connections:
- net Net-(J8-Pad2) renamed /P_FPGA_3V3
- net Net-(J9-Pad2) renamed /V_FPGA_3V3
- C1 pad 1: /V_5V -> Net-(C1-Pad1)
- C13 pad 1: +5V -> +5VA
- C14 pad 1: +5V -> +5VL
- C17 pad 1: Net-(C17-Pad1) -> +5V
- C2 pad 1: /P_5V -> Net-(C2-Pad1)
- C22 pad 1: /V_3V3_2 -> /VDRV_LDO_3V3
- C24 pad 1: /V_3V3_1 -> /VREF_LDO_3V3
- C25 pad 1: /P_3V3_2 -> /PDRV_LDO_3V3
- C26 pad 1: /P_3V3_1 -> /PREF_LDO_3V3
- C3 pad 1: /V_5V -> Net-(C1-Pad1)
- C4 pad 1: /V_5V -> Net-(C1-Pad1)
- C5 pad 1: /P_5V -> Net-(C2-Pad1)
- C6 pad 1: /P_5V -> Net-(C2-Pad1)
- C7 pad 1: +5V -> +5VA
- C8 pad 1: +5V -> +5VL
- D1 pad 1: Net-(C17-Pad1) -> +5V
- D1 pad 2: Net-(D1-Pad2) -> Net-(C18-Pad1)
- F1 pad 1: +5V -> Net-(C18-Pad1)
- F1 pad 2: Net-(C17-Pad1) -> Net-(F1-Pad2)
- FB1 pad 1: +5V -> +5VA
- FB1 pad 2: /V_5V -> Net-(C1-Pad1)
- FB2 pad 1: +5V -> +5VL
- FB2 pad 2: /P_5V -> Net-(C2-Pad1)
- FB7 pad 2: +5V -> +5VA
- FB8 pad 2: +5V -> +5VL
- J1 pad 1: GND -> /V_DRIVE_P
- J1 pad 10: /V_3V3_2 -> /V_SENSE_N
- J1 pad 11: /V_SENSE_P -> /VSNS_3V3
- J1 pad 12: /V_SENSE_N -> GND
- J1 pad 2: /V_5V -> /V_DRIVE_N
- J1 pad 3: /V_DRIVE_P -> /VDRV_3V3
- J1 pad 4: /V_DRIVE_N -> GND
- J1 pad 5: GND -> /V_REF_P
- J1 pad 6: /V_3V3_1 -> /V_REF_N
- J1 pad 7: /V_REF_P -> /VREF_3V3
- J1 pad 8: /V_REF_N -> GND
- J1 pad 9: GND -> /V_SENSE_P
- J2 pad 1: GND -> /P_DRIVE_P
- J2 pad 10: /P_3V3_2 -> /P_SENSE_N
- J2 pad 11: /P_SENSE_P -> /PSNS_3V3
- J2 pad 12: /P_SENSE_N -> GND
- J2 pad 2: /P_5V -> /P_DRIVE_N
- J2 pad 3: /P_DRIVE_P -> /PDRV_3V3
- J2 pad 4: /P_DRIVE_N -> GND
- J2 pad 5: GND -> /P_REF_P
- J2 pad 6: /P_3V3_1 -> /P_REF_N
- J2 pad 7: /P_REF_P -> /PREF_3V3
- J2 pad 8: /P_REF_N -> GND
- J2 pad 9: GND -> /P_SENSE_P
- J3 pad 1: Net-(D1-Pad2) -> Net-(F1-Pad2)
- U10 pad 1: /P_5V -> Net-(C2-Pad1)
- U10 pad 3: /P_5V -> Net-(C2-Pad1)
- U10 pad 5: /P_3V3_1 -> /PREF_LDO_3V3
- U7 pad 1: /V_5V -> Net-(C1-Pad1)
- U7 pad 3: /V_5V -> Net-(C1-Pad1)
- U7 pad 5: /V_3V3_2 -> /VDRV_LDO_3V3
- U8 pad 1: /V_5V -> Net-(C1-Pad1)
- U8 pad 3: /V_5V -> Net-(C1-Pad1)
- U8 pad 5: /V_3V3_1 -> /VREF_LDO_3V3
- U9 pad 1: /P_5V -> Net-(C2-Pad1)
- U9 pad 3: /P_5V -> Net-(C2-Pad1)
- U9 pad 5: /P_3V3_2 -> /PDRV_LDO_3V3
Routing:
- net GND: track 0.00 -> 72.9 mm
- net /P_FPGA_3V3: track 0.00 -> 52.9 mm
- net /V_FPGA_3V3: track 0.00 -> 52.2 mm
- net /P_SENSE_P: track 0.00 -> 39.1 mm
- net /V_SENSE_P: track 0.00 -> 38.1 mm
- net /P_SENSE_N: track 0.00 -> 37.3 mm
- net /V_SENSE_N: track 0.00 -> 37.0 mm
- net /V_REF_P: track 0.00 -> 32.2 mm
- net /P_REF_P: track 0.00 -> 32.2 mm
- net /P_DRIVE_P: track 0.00 -> 31.5 mm
- net /V_DRIVE_P: track 0.00 -> 31.5 mm
- net /V_REF_N: track 0.00 -> 31.2 mm
- net /SPI_MOSI: track 0.00 -> 31.0 mm
- net /SPI_MISO: track 0.00 -> 31.0 mm
- net /I2S_MCLK: track 0.00 -> 31.0 mm
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Other:
- board size 199.4 x 61 mm -> 209.6 x 61 mm

Commit message: teensytheremin fpga main board kicad project
Parts:
- moved J6 15.3 mm to (95.2, 111.5)
- moved J7 10.1 mm to (108.0, 100.1)
- moved C2 5.68 mm to (199.4, 63.5)
- moved C8 5.68 mm to (194.3, 63.5)
- moved FB2 5.68 mm to (196.8, 68.6)
- moved C14 3.81 mm to (178.1, 99.1)
- moved C16 3.81 mm to (182.6, 99.1)
- moved FB8 3.81 mm to (179.1, 104.1)
- moved J1 2.84 mm to (48.3, 99.1)
- moved J2 2.54 mm to (233.7, 71.1)
- moved J10 1.80 mm to (111.8, 63.5)
- moved C28 1.27 mm to (85.1, 123.2)
- moved C3 1.27 mm to (76.5, 95.2)
- moved C4 1.27 mm to (76.5, 102.9)
- moved J4 1.27 mm to (180.3, 70.1)
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Routing:
- net /V_DRIVE_P: track 31.5 -> 34.0 mm
- net /V_REF_N: track 31.2 -> 33.7 mm
- net /V_DRIVE_N: track 24.6 -> 27.2 mm
- net /V_SENSE_N: track 37.0 -> 39.6 mm
- net /V_REF_P: track 32.2 -> 34.8 mm
- net /P_SENSE_N: track 37.3 -> 39.9 mm
- net /P_SENSE_P: track 39.1 -> 41.7 mm
- net /P_REF_P: track 32.2 -> 34.8 mm
- net /P_REF_N: track 30.4 -> 33.0 mm
- net /P_DRIVE_P: track 31.5 -> 34.0 mm
- net /P_DRIVE_N: track 24.6 -> 27.2 mm
- net /V_SENSE_P: track 38.1 -> 40.6 mm
- net /VREF_3V3: track 15.8 -> 16.8 mm
- net /PREF_3V3: track 15.8 -> 16.8 mm
- net /VDRV_3V3: track 19.4 -> 20.4 mm
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Other:
- board size 209.6 x 61 mm -> 210.8 x 61 mm

Commit message: update preadme; convert pcb schematic to KiCAD 6.0
Parts:
- removed C1, C13, C14, C2: 10uF, Capacitor_SMD:C_0805_2012Metric
- removed FB1, FB2, FB7, FB8: 680uH, Inductor_SMD:L_1812_4532Metric
- added SW1: SW_Push, Button_Switch_THT:SW_Tactile_SPST_Angled_PTS645Vx58-2LFS, F.Cu at (109.8, 57.4)
- C15, C16: value 10uF -> 2.2uF
- moved D5 79.6 mm to (112.5, 75.5), turned to 180 degrees
- moved D3 77.3 mm to (111.8, 68.6), turned to 90 degrees
- moved D4 74.1 mm to (100.9, 75.5)
- moved D2 71.9 mm to (101.6, 68.6), turned to 90 degrees
- moved D1 67.6 mm to (106.7, 68.6), turned to 90 degrees
- moved C27 62.5 mm to (115.6, 71.3), turned to 90 degrees
- moved C18 59.4 mm to (97.8, 67.8), turned to -90 degrees
- moved C28 53.1 mm to (97.8, 71.7), turned to 90 degrees
- moved C7 26.0 mm to (83.8, 92.4)
- moved J10 20.1 mm to (92.7, 57.1)
- moved F1 15.6 mm to (131.9, 71.1)
- moved C16 15.5 mm to (189.2, 113.0), turned to 180 degrees
- moved C15 13.6 mm to (91.1, 66.0), turned to 0 degrees
- moved C17 5.08 mm to (106.7, 75.2), turned to -90 degrees
- moved C8 4.41 mm to (198.1, 65.7)
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Connections:
- net Net-(C18-Pad1) renamed /+5V_F
- net Net-(F1-Pad2) renamed /+5V_IN
- C15 pad 1: /V_FPGA_5V -> +5VA
- C16 pad 1: /P_FPGA_5V -> +5VL
- C29 pad 1: Net-(C1-Pad1) -> +5VA
- C3 pad 1: Net-(C1-Pad1) -> +5VA
- C30 pad 1: Net-(C2-Pad1) -> +5VL
- C4 pad 1: Net-(C1-Pad1) -> +5VA
- C5 pad 1: Net-(C2-Pad1) -> +5VL
- C6 pad 1: Net-(C2-Pad1) -> +5VL
- U1 pad 11: Net-(U1-Pad11) -> unconnected-(U1-Pad11)
- U1 pad 15: Net-(U1-Pad15) -> +3V3
- U1 pad 16: Net-(U1-Pad16) -> /P_DONE
- U1 pad 17: Net-(U1-Pad17) -> /P_RECONFIG_N
- U1 pad 18: Net-(U1-Pad18) -> /PED1
- U1 pad 19: Net-(U1-Pad19) -> unconnected-(U1-Pad19)
- U1 pad 2: Net-(U1-Pad2) -> unconnected-(U1-Pad2)
- U1 pad 20: Net-(U1-Pad20) -> unconnected-(U1-Pad20)
- U1 pad 21: Net-(U1-Pad21) -> unconnected-(U1-Pad21)
- U1 pad 22: Net-(U1-Pad22) -> unconnected-(U1-Pad22)
- U1 pad 23: Net-(U1-Pad23) -> unconnected-(U1-Pad23)
- U1 pad 24: Net-(U1-Pad24) -> unconnected-(U1-Pad24)
- U1 pad 25: Net-(U1-Pad25) -> /V_RECONFIG_N
- U1 pad 26: Net-(U1-Pad26) -> /V_DONE
- U1 pad 27: Net-(U1-Pad27) -> unconnected-(U1-Pad27)
- U1 pad 28: Net-(U1-Pad28) -> /SPI_V_CS
- U1 pad 29: Net-(U1-Pad29) -> /SPI_P_CS
- U1 pad 3: Net-(U1-Pad3) -> unconnected-(U1-Pad3)
- U1 pad 30: Net-(U1-Pad30) -> unconnected-(U1-Pad30)
- U1 pad 31: Net-(U1-Pad31) -> unconnected-(U1-Pad31)
- U1 pad 32: Net-(U1-Pad32) -> unconnected-(U1-Pad32)
- U1 pad 33: Net-(U1-Pad33) -> unconnected-(U1-Pad33)
- U1 pad 4: Net-(U1-Pad4) -> unconnected-(U1-Pad4)
- U1 pad 44: Net-(U1-Pad44) -> unconnected-(U1-Pad44)
- U1 pad 49: Net-(U1-Pad49) -> unconnected-(U1-Pad49)
- U1 pad 5: Net-(U1-Pad5) -> unconnected-(U1-Pad5)
- U1 pad 50: Net-(U1-Pad50) -> unconnected-(U1-Pad50)
- U1 pad 51: Net-(U1-Pad51) -> unconnected-(U1-Pad51)
- U1 pad 53: Net-(U1-Pad53) -> unconnected-(U1-Pad53)
- U1 pad 6: Net-(U1-Pad6) -> unconnected-(U1-Pad6)
- U1 pad 7: Net-(U1-Pad7) -> unconnected-(U1-Pad7)
- U1 pad 8: /SPI_A_MEMCS -> /I2S_FPGA_OUT
- U10 pad 1: Net-(C2-Pad1) -> +5VL
- U10 pad 3: Net-(C2-Pad1) -> +5VL
- U11 pad 1: Net-(C1-Pad1) -> +5VA
- U11 pad 3: Net-(C1-Pad1) -> +5VA
- U12 pad 1: Net-(C2-Pad1) -> +5VL
- U12 pad 3: Net-(C2-Pad1) -> +5VL
- U2 pad 17: Net-(U2-Pad17) -> unconnected-(U2-Pad17)
- U2 pad 39: Net-(U2-Pad39) -> unconnected-(U2-Pad39)
- U2 pad 40: Net-(U2-Pad40) -> unconnected-(U2-Pad40)
- U2 pad 8: /SPI_A_MEMCS -> unconnected-(U2-Pad8)
- U3 pad 11: Net-(U3-Pad11) -> unconnected-(U3-Pad11)
- U3 pad 15: Net-(U3-Pad15) -> unconnected-(U3-Pad15)
- U3 pad 20: Net-(U3-Pad20) -> unconnected-(U3-Pad20)
- U3 pad 21: Net-(U3-Pad21) -> unconnected-(U3-Pad21)
- U3 pad 22: /V_FPGA_5V -> +5VA
- U3 pad 23: /V_FPGA_5V -> +5VA
- U3 pad 24: Net-(U3-Pad24) -> unconnected-(U3-Pad24)
- U3 pad 25: Net-(U3-Pad25) -> unconnected-(U3-Pad25)
- U3 pad 26: Net-(U3-Pad26) -> unconnected-(U3-Pad26)
- U3 pad 27: Net-(U3-Pad27) -> unconnected-(U3-Pad27)
- U3 pad 28: Net-(U3-Pad28) -> unconnected-(U3-Pad28)
- U3 pad 29: Net-(U3-Pad29) -> unconnected-(U3-Pad29)
- U3 pad 3: Net-(U3-Pad3) -> unconnected-(U3-Pad3)
- U3 pad 33: Net-(U3-Pad33) -> unconnected-(U3-Pad33)
- U3 pad 34: Net-(U3-Pad34) -> unconnected-(U3-Pad34)
- U3 pad 35: Net-(U3-Pad35) -> unconnected-(U3-Pad35)
- U3 pad 36: Net-(U3-Pad36) -> unconnected-(U3-Pad36)
- U3 pad 4: Net-(U3-Pad4) -> unconnected-(U3-Pad4)
- U4 pad 11: Net-(U4-Pad11) -> unconnected-(U4-Pad11)
- U4 pad 15: Net-(U4-Pad15) -> unconnected-(U4-Pad15)
- U4 pad 20: Net-(U4-Pad20) -> unconnected-(U4-Pad20)
- U4 pad 21: Net-(U4-Pad21) -> unconnected-(U4-Pad21)
- U4 pad 22: /P_FPGA_5V -> +5VL
- U4 pad 23: /P_FPGA_5V -> +5VL
- U4 pad 24: Net-(U4-Pad24) -> unconnected-(U4-Pad24)
- U4 pad 25: Net-(U4-Pad25) -> unconnected-(U4-Pad25)
- U4 pad 26: Net-(U4-Pad26) -> unconnected-(U4-Pad26)
- U4 pad 27: Net-(U4-Pad27) -> unconnected-(U4-Pad27)
- U4 pad 28: Net-(U4-Pad28) -> unconnected-(U4-Pad28)
- U4 pad 29: Net-(U4-Pad29) -> unconnected-(U4-Pad29)
- U4 pad 3: Net-(U4-Pad3) -> unconnected-(U4-Pad3)
- U4 pad 33: Net-(U4-Pad33) -> unconnected-(U4-Pad33)
- U4 pad 34: Net-(U4-Pad34) -> unconnected-(U4-Pad34)
- U4 pad 35: Net-(U4-Pad35) -> unconnected-(U4-Pad35)
- U4 pad 36: Net-(U4-Pad36) -> unconnected-(U4-Pad36)
- U4 pad 4: Net-(U4-Pad4) -> unconnected-(U4-Pad4)
- U7 pad 1: Net-(C1-Pad1) -> +5VA
- U7 pad 3: Net-(C1-Pad1) -> +5VA
- U8 pad 1: Net-(C1-Pad1) -> +5VA
- U8 pad 3: Net-(C1-Pad1) -> +5VA
- U9 pad 1: Net-(C2-Pad1) -> +5VL
- U9 pad 3: Net-(C2-Pad1) -> +5VL
Routing:
- net /SDA: track 0.00 -> 31.0 mm
- net /SCL: track 0.00 -> 31.0 mm
- net +3V3: track 0.00 -> 31.0 mm
Other:
- net class Default removed
